File: hardware/jlink-adapter.kicad_sch (KiCad schematic)
At the start: 37 parts, among them J1 EZmate-4, J2 Conn_02x05_Odd_Even, J3 Conn_02x10_Odd_Even, J4 TC2030-IDC-NL, SW1 SW_Push, SW2 SW_Push, U1 TPS7A0333DBVR, U2 TPS7A0333DBVR, U4 TPS7A0333DBVR, U5 STM32C011F6Ux

Commit message: hw: fix led r values
Parts:
- R1, R4, R7, R8, R9: value 1k -> 220
Changed lines of the file:
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@@
 			)
 		)
-		(property "Value" "1k"
+		(property "Value" "220"
 			(at 236.22 149.8599 0)
 			(effects
@@
 			)
 		)
-		(property "Value" "1k"
+		(property "Value" "220"
 			(at 224.79 149.8599 0)
 			(effects
@@
 			)
 		)
-		(property "Value" "1k"
+		(property "Value" "220"
 			(at 247.65 149.8599 0)
 			(effects
@@
 			)
 		)
-		(property "Value" "1k"
+		(property "Value" "220"
 			(at 259.08 149.8599 0)
 			(effects
@@
 			)
 		)
-		(property "Value" "1k"
+		(property "Value" "220"
 			(at 270.51 149.8599 0)
 			(effects
