File: hardware/jlink-adapter.kicad_sch (KiCad schematic)
At the start: 37 parts, among them J1 EZmate-4, J2 Conn_02x05_Odd_Even, J3 Conn_02x10_Odd_Even, J4 TC2030-IDC-NL, SW1 SW_Push, SW2 SW_Push, U1 TPS7A0333DBVR, U2 TPS7A0333DBVR, U4 TPS7A0333DBVR, U5 STM32C011F6Ux

Commit message: hw: use lower output caps
Parts:
- C2, C4: value 10u -> 100n
Changed lines of the file:
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@@
 		(fields_autoplaced yes)
 		(property "Reference" "C4"
-			(at 64.77 135.89 0)
+			(at 64.77 135.8899 0)
 			(effects
 				(font
@@
 			)
 		)
-		(property "Value" "10u"
-			(at 64.77 138.43 0)
+		(property "Value" "100n"
+			(at 64.77 138.4299 0)
 			(effects
 				(font
@@
 		(fields_autoplaced yes)
 		(property "Reference" "C2"
-			(at 64.77 91.44 0)
+			(at 64.77 91.4399 0)
 			(effects
 				(font
@@
 			)
 		)
-		(property "Value" "10u"
-			(at 64.77 93.98 0)
-			(effects
-				(font
+		(property "Value" "100n"
+			(at 64.77 93.9799 0)
+			(effects
+				(font

Commit message: hw: add note about reverse diodes
Other:
- note added: "TODO: diodes"
Changed lines of the file:
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@@
+		)
+	)
+	(text "TODO: diodes"
+		(exclude_from_sim no)
+		(at 25.4 83.82 0)
+		(effects
+			(font
+				(size 1.27 1.27)
+			)
 		)
 	)
@@
 		)
 	)
+	(text "TODO: diodes"
+		(exclude_from_sim no)
+		(at 26.67 128.27 0)
+		(effects
+			(font
+				(size 1.27 1.27)
+			)
+		)
+	)

Commit message: hw: assembly fixes
Parts:
- U1: value TPS7A0333DBVR -> TPS7A0318DBVR
Connections:
- net EN_1V8: now also R3.1, U1.3 (EN), U5.13 (PA8); no longer R2.1, U2.3 (EN), U5.14 (PA9/PA11)
- net EN_3V3: now also R2.1, U2.3 (EN), U5.14 (PA9/PA11); no longer R3.1, U1.3 (EN), U5.13 (PA8)
Changed lines of the file:
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@@
 	(text "3.3V LDO"
 		(exclude_from_sim no)
+		(at 15.24 118.11 0)
+		(effects
+			(font
+				(size 3 3)
+			)
+			(justify left bottom)
+		)
+	)
+	(text "TODO: diodes"
+		(exclude_from_sim no)
+		(at 25.4 83.82 0)
+		(effects
+			(font
+				(size 1.27 1.27)
+			)
+		)
+	)
+	(text "3.3V LDO (system)"
+		(exclude_from_sim no)
+		(at 97.79 20.32 0)
+		(effects
+			(font
+				(size 3 3)
+			)
+			(justify left bottom)
+		)
+	)
+	(text "VCOM-TX"
+		(exclude_from_sim no)
+		(at 49.53 36.83 0)
+		(effects
+			(font
+				(size 1.27 1.27)
+			)
+			(justify left bottom)
+		)
+	)
+	(text "GND"
+		(exclude_from_sim no)
+		(at 58.42 181.61 0)
+		(effects
+			(font
+				(size 1.27 1.27)
+			)
+			(justify right bottom)
+		)
+	)
+	(text "TCK"
+		(exclude_from_sim no)
+		(at 60.96 41.91 0)
+		(effects
+			(font
+				(size 1.27 1.27)
+			)
+			(justify left bottom)
+		)
+	)
+	(text "VCC"
+		(exclude_from_sim no)
+		(at 223.52 92.71 0)
+		(effects
+			(font
+				(size 1.27 1.27)
+			)
+			(justify right bottom)
+		)
+	)
+	(text "1.8V LDO"
+		(exclude_from_sim no)
 		(at 15.24 73.66 0)
-		(effects
-			(font
-				(size 3 3)
-			)
-			(justify left bottom)
-		)
-	)
-	(text "TODO: diodes"
-		(exclude_from_sim no)
-		(at 25.4 83.82 0)
-		(effects
-			(font
-				(size 1.27 1.27)
-			)
-		)
-	)
-	(text "3.3V LDO (system)"
-		(exclude_from_sim no)
-		(at 97.79 20.32 0)
-		(effects
-			(font
-				(size 3 3)
-			)
-			(justify left bottom)
-		)
-	)
-	(text "VCOM-TX"
-		(exclude_from_sim no)
-		(at 49.53 36.83 0)
-		(effects
-			(font
-				(size 1.27 1.27)
-			)
-			(justify left bottom)
-		)
-	)
-	(text "GND"
-		(exclude_from_sim no)
-		(at 58.42 181.61 0)
-		(effects
-			(font
-				(size 1.27 1.27)
-			)
-			(justify right bottom)
-		)
-	)
-	(text "TCK"
-		(exclude_from_sim no)
-		(at 60.96 41.91 0)
-		(effects
-			(font
-				(size 1.27 1.27)
-			)
-			(justify left bottom)
-		)
-	)
-	(text "VCC"
-		(exclude_from_sim no)
-		(at 223.52 92.71 0)
-		(effects
-			(font
-				(size 1.27 1.27)
-			)
-			(justify right bottom)
-		)
-	)
-	(text "1.8V LDO"
-		(exclude_from_sim no)
-		(at 15.24 118.11 0)
 		(effects
 			(font
@@
 	)
 	(label "EN_3V3"
-		(at 261.62 50.8 180)
+		(at 261.62 53.34 180)
 		(fields_autoplaced yes)
 		(effects
@@
 		)
 	)
-	(label "EN_1V8"
+	(label "EN_3V3"
 		(at 24.13 133.35 0)
 		(fields_autoplaced yes)
@@
 	)
 	(label "EN_1V8"
-		(at 261.62 53.34 180)
+		(at 261.62 50.8 180)
 		(fields_autoplaced yes)
 		(effects
@@
 		)
 	)
-	(label "EN_3V3"
+	(label "EN_1V8"
 		(at 24.13 88.9 0)
 		(fields_autoplaced yes)
@@
 			)
 		)
-		(property "Value" "TPS7A0333DBVR"
+		(property "Value" "TPS7A0318DBVR"
 			(at 48.26 81.28 0)
 			(effects
