File: hardware/jlink-adapter.kicad_pcb (KiCad board)
At the start: 2 copper layers, 26 x 27 mm, 38 parts, among them J1 EZmate-4, J2 Conn_02x05_Odd_Even, J3 Conn_02x10_Odd_Even, J4 TC2030-IDC-NL, SW1 SW_Push, SW2 SW_Push, U1 TPS7A0333DBVR, U2 TPS7A0333DBVR, U4 TPS7A0333DBVR, U5 STM32C011F6Ux

Commit message: hw: fix led r values
Parts:
- R1, R4, R7, R8, R9: value 1k -> 220
Changed lines of the file:
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@@
 			)
 		)
-		(property "Value" "1k"
+		(property "Value" "220"
 			(at 0 -1.1 -90)
 			(unlocked yes)
@@
 			)
 		)
-		(property "Value" "1k"
+		(property "Value" "220"
 			(at 0 -1.1 -90)
 			(unlocked yes)
@@
 			)
 		)
-		(property "Value" "1k"
+		(property "Value" "220"
 			(at 0 -1.1 -90)
 			(unlocked yes)
@@
 			)
 		)
-		(property "Value" "1k"
+		(property "Value" "220"
 			(at 0 -1.1 -90)
 			(unlocked yes)
@@
 			)
 		)
-		(property "Value" "1k"
+		(property "Value" "220"
 			(at 0 -1.1 -90)
 			(unlocked yes)

Commit message: hw: assembly fixes
Parts:
- C2, C4: value 10u -> 100n
- U1: value TPS7A0333DBVR -> TPS7A0318DBVR
Connections:
- R2 pad 1: /EN_1V8 -> /EN_3V3
- R3 pad 1: /EN_3V3 -> /EN_1V8
- U1 pad 3: /EN_3V3 -> /EN_1V8
- U2 pad 3: /EN_1V8 -> /EN_3V3
- U5 pad 13: /EN_3V3 -> /EN_1V8
- U5 pad 14: /EN_1V8 -> /EN_3V3
Routing:
- net /EN_3V3: track 15.3 -> 11.0 mm
- net /EN_1V8: track 11.0 -> 15.3 mm
Changed lines of the file:
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@@
 		(pad_to_mask_clearance 0)
 		(allow_soldermask_bridges_in_footprints no)
+		(aux_axis_origin 149 123)
 		(pcbplotparams
 			(layerselection 0x00010fc_ffffffff)
@@
 			(size 0.7 0.3)
 			(layers "F.Cu" "F.Paste" "F.Mask")
-			(net 35 "/EN_3V3")
+			(net 34 "/EN_1V8")
 			(pinfunction "PA8")
 			(pintype "bidirectional")
@@
 			(size 0.7 0.3)
 			(layers "F.Cu" "F.Paste" "F.Mask")
-			(net 34 "/EN_1V8")
+			(net 35 "/EN_3V3")
 			(pinfunction "PA9/PA11")
 			(pintype "bidirectional")
@@
 			(layers "F.Cu" "F.Paste" "F.Mask")
 			(roundrect_rratio 0.25)
-			(net 34 "/EN_1V8")
+			(net 35 "/EN_3V3")
 			(pintype "passive")
 		)
@@
 			)
 		)
-		(property "Value" "10u"
+		(property "Value" "100n"
 			(at 0 1.43 0)
 			(layer "F.Fab")
@@
 			)
 		)
-		(property "Value" "TPS7A0333DBVR"
+		(property "Value" "TPS7A0318DBVR"
 			(at 0 2.4 90)
 			(layer "F.Fab")
@@
 			(layers "F.Cu" "F.Paste" "F.Mask")
 			(roundrect_rratio 0.25)
-			(net 35 "/EN_3V3")
+			(net 34 "/EN_1V8")
 			(pinfunction "EN")
 			(pintype "input")
@@
 			(layers "F.Cu" "F.Paste" "F.Mask")
 			(roundrect_rratio 0.25)
-			(net 34 "/EN_1V8")
+			(net 35 "/EN_3V3")
 			(pinfunction "EN")
 			(pintype "input")
@@
 			)
 		)
-		(property "Value" "10u"
+		(property "Value" "100n"
 			(at 0 1.43 0)
 			(layer "F.Fab")
@@
 			(layers "F.Cu" "F.Paste" "F.Mask")
 			(roundrect_rratio 0.25)
-			(net 35 "/EN_3V3")
+			(net 34 "/EN_1V8")
 			(pintype "passive")
 		)
@@
 	)
 	(segment
-		(start 156.9 101.8)
-		(end 156.1 102.6)
+		(start 170.45 102.1625)
+		(end 169.8625 102.1625)
 		(width 0.2)
 		(layer "F.Cu")
@@
 	)
 	(segment
-		(start 165.1 101.8)
-		(end 164.4 101.8)
+		(start 169.8625 102.1625)
+		(end 169.5 101.8)
 		(width 0.2)
 		(layer "F.Cu")
@@
 	)
 	(segment
-		(start 159.8 101.8)
-		(end 156.9 101.8)
+		(start 169.5 101.8)
+		(end 168.8 101.8)
 		(width 0.2)
 		(layer "F.Cu")
@@
 	)
 	(segment
-		(start 166.05 102.1625)
-		(end 165.4625 102.1625)
+		(start 159.8 102.6)
+		(end 159.4 102.2)
 		(width 0.2)
 		(layer "F.Cu")
@@
 	)
 	(segment
-		(start 156.1 102.6)
-		(end 156.1 103.2)
+		(start 157 102.2)
+		(end 156.6 102.6)
 		(width 0.2)
 		(layer "F.Cu")
@@
 	)
 	(segment
-		(start 165.4625 102.1625)
-		(end 165.1 101.8)
+		(start 156.6 102.6)
+		(end 156.6 103.2)
+		(width 0.2)
+		(layer "F.Cu")
+		(net 34)
+	)
+	(segment
+		(start 159.4 102.2)
+		(end 157 102.2)
 		(width 0.2)
 		(layer "F.Cu")
@@
 	)
 	(via
-		(at 159.8 101.8)
+		(at 159.8 102.6)
 		(size 0.45)
 		(drill 0.2)
@@
 	)
 	(via
-		(at 164.4 101.8)
+		(at 168.8 101.8)
 		(size 0.45)
 		(drill 0.2)
@@
 	)
 	(segment
-		(start 159.8 101.8)
-		(end 164.4 101.8)
+		(start 159.8 102.6)
+		(end 160.1 102.3)
 		(width 0.2)
 		(layer "B.Cu")
@@
 	)
 	(segment
-		(start 170.45 102.1625)
-		(end 169.8625 102.1625)
+		(start 160.1 102.3)
+		(end 164.6 102.3)
 		(width 0.2)
-		(layer "F.Cu")
-		(net 35)
+		(layer "B.Cu")
+		(net 34)
 	)
 	(segment
-		(start 169.8625 102.1625)
-		(end 169.5 101.8)
+		(start 165.1 101.8)
+		(end 168.8 101.8)
+		(width 0.2)
+		(layer "B.Cu")
+		(net 34)
+	)
+	(segment
+		(start 164.6 102.3)
+		(end 165.1 101.8)
+		(width 0.2)
+		(layer "B.Cu")
+		(net 34)
+	)
+	(segment
+		(start 156.9 101.8)
+		(end 156.1 102.6)
 		(width 0.2)
 		(layer "F.Cu")
@@
 	)
 	(segment
-		(start 169.5 101.8)
-		(end 168.8 101.8)
+		(start 165.1 101.8)
+		(end 164.4 101.8)
 		(width 0.2)
 		(layer "F.Cu")
@@
 	)
 	(segment
-		(start 159.8 102.6)
-		(end 159.4 102.2)
+		(start 159.8 101.8)
+		(end 156.9 101.8)
 		(width 0.2)
 		(layer "F.Cu")
@@
 	)
 	(segment
-		(start 157 102.2)
-		(end 156.6 102.6)
+		(start 166.05 102.1625)
+		(end 165.4625 102.1625)
 		(width 0.2)
 		(layer "F.Cu")
@@
 	)
 	(segment
-		(start 156.6 102.6)
-		(end 156.6 103.2)
+		(start 156.1 102.6)
+		(end 156.1 103.2)
 		(width 0.2)
 		(layer "F.Cu")
@@
 	)
 	(segment
-		(start 159.4 102.2)
-		(end 157 102.2)
+		(start 165.4625 102.1625)
+		(end 165.1 101.8)
 		(width 0.2)
 		(layer "F.Cu")
@@
 	)
 	(via
-		(at 159.8 102.6)
+		(at 159.8 101.8)
 		(size 0.45)
 		(drill 0.2)
@@
 	)
 	(via
-		(at 168.8 101.8)
+		(at 164.4 101.8)
 		(size 0.45)
 		(drill 0.2)
@@
 	)
 	(segment
-		(start 159.8 102.6)
-		(end 160.1 102.3)
-		(width 0.2)
-		(layer "B.Cu")
-		(net 35)
-	)
-	(segment
-		(start 160.1 102.3)
-		(end 164.6 102.3)
-		(width 0.2)
-		(layer "B.Cu")
-		(net 35)
-	)
-	(segment
-		(start 165.1 101.8)
-		(end 168.8 101.8)
-		(width 0.2)
-		(layer "B.Cu")
-		(net 35)
-	)
-	(segment
-		(start 164.6 102.3)
-		(end 165.1 101.8)
+		(start 159.8 101.8)
+		(end 164.4 101.8)
 		(width 0.2)
 		(layer "B.Cu")
